Commit message: testando

File: description/robot.urdf.xacro (robot description, xacro)
@@ -3,5 +3,5 @@
   xmlns:xacro="http://ros.org/wiki/xacro">
   <!-- Definicao de Algumas Contantes -->
-  <xacro:property name="base_width" value="0.31"/> <!-- Largura da base -->
+  <xacro:property name="base_width" value="0.21"/> <!-- Largura da base -->
   <xacro:property name="base_length" value="0.42"/> <!-- Comprimento da base -->
   <xacro:property name="base_height" value="0.18"/> <!-- Altura da base -->

Commit message: correct odometry

File: description/robot.urdf.xacro (robot description, xacro)
@@ -2,14 +2,14 @@
 <robot name="prm_robot"
   xmlns:xacro="http://ros.org/wiki/xacro">
-  <!-- Definicao de Algumas Contantes -->
-  <xacro:property name="base_width" value="0.31"/> <!-- Largura da base -->
-  <xacro:property name="base_length" value="0.42"/> <!-- Comprimento da base -->
-  <xacro:property name="base_height" value="0.18"/> <!-- Altura da base -->
-  <xacro:property name="wheel_radius" value="0.10"/> <!-- Raio da roda -->
-  <xacro:property name="wheel_width" value="0.04"/> <!-- Largura da roda -->
-  <xacro:property name="wheel_ygap" value="0.025"/> <!-- Distancia entre as rodas -->
-  <xacro:property name="wheel_zoff" value="0.05"/> <!-- Deslocamento da roda em Z -->
-  <xacro:property name="wheel_xoff" value="0.12"/> <!-- Deslocamento da roda em X -->
-  <xacro:property name="caster_xoff" value="0.14"/> <!-- Deslocamento do caster em X -->
+  <!-- Definição de algumas constantes (comprimento e largura reduzidos pela metade, altura mantida) -->
+  <xacro:property name="base_width" value="0.155"/> <!-- Largura da base (original 0.31 reduzido para 0.155) -->
+  <xacro:property name="base_length" value="0.21"/> <!-- Comprimento da base (original 0.42 reduzido para 0.21) -->
+  <xacro:property name="base_height" value="0.18"/> <!-- Altura da base (permanece 0.18) -->
+  <xacro:property name="wheel_radius" value="0.10"/> <!-- Raio da roda (permanece 0.10) -->
+  <xacro:property name="wheel_width" value="0.04"/>  <!-- Largura da roda (permanece 0.04) -->
+  <xacro:property name="wheel_ygap" value="0.0125"/> <!-- Distância entre as rodas em Y (original 0.025 reduzido para 0.0125) -->
+  <xacro:property name="wheel_zoff" value="0.05"/>   <!-- Deslocamento da roda em Z (permanece 0.05) -->
+  <xacro:property name="wheel_xoff" value="0.06"/>   <!-- Deslocamento da roda em X (original 0.12 reduzido para 0.06) -->
+  <xacro:property name="caster_xoff" value="0.07"/> <!-- Deslocamento do caster em X (original 0.14 reduzido para 0.07) -->
   <!-- Definição de algumas propriedades inerciais -->
   <xacro:macro name="box_inertia" params="m w h d">
@@ -17,12 +17,16 @@
       <origin xyz="0 0 0" rpy="${pi/2} 0 ${pi/2}"/>
       <mass value="${m}"/>
-      <inertia ixx="${(m/12) * (h*h + d*d)}" ixy="0.0" ixz="0.0" iyy="${(m/12) * (w*w + d*d)}" iyz="0.0" izz="${(m/12) * (w*w + h*h)}"/>
+      <inertia ixx="${(m/12) * (h*h + d*d)}" ixy="0.0" ixz="0.0"
+               iyy="${(m/12) * (w*w + d*d)}" iyz="0.0"
+               izz="${(m/12) * (w*w + h*h)}"/>
     </inertial>
   </xacro:macro>
   <xacro:macro name="cylinder_inertia" params="m r h">
     <inertial>
-      <origin xyz="0 0 0" rpy="${pi/2} 0 0" />
+      <origin xyz="0 0 0" rpy="${pi/2} 0 0"/>
       <mass value="${m}"/>
-      <inertia ixx="${(m/12) * (3*r*r + h*h)}" ixy = "0" ixz = "0" iyy="${(m/12) * (3*r*r + h*h)}" iyz = "0" izz="${(m/2) * (r*r)}"/>
+      <inertia ixx="${(m/12) * (3*r*r + h*h)}" ixy="0" ixz="0"
+               iyy="${(m/12) * (3*r*r + h*h)}" iyz="0"
+               izz="${(m/2) * (r*r)}"/>
     </inertial>
   </xacro:macro>
@@ -30,10 +34,13 @@
     <inertial>
       <mass value="${m}"/>
-      <inertia ixx="${(2/5) * m * (r*r)}" ixy="0.0" ixz="0.0" iyy="${(2/5) * m * (r*r)}" iyz="0.0" izz="${(2/5) * m * (r*r)}"/>
+      <inertia ixx="${(2/5) * m * (r*r)}" ixy="0.0" ixz="0.0"
+               iyy="${(2/5) * m * (r*r)}" iyz="0.0"
+               izz="${(2/5) * m * (r*r)}"/>
     </inertial>
   </xacro:macro>
-  <!-- Definindo plugin para publiar a pose do robo -->
+  <!-- Plugin do Gazebo/Ignition para publicar pose do robô -->
   <gazebo>
-    <plugin filename="libignition-gazebo-pose-publisher-system" name="ignition::gazebo::systems::PosePublisher">
+    <plugin filename="libignition-gazebo-pose-publisher-system"
+            name="ignition::gazebo::systems::PosePublisher">
       <publish_link_pose>false</publish_link_pose>
       <publish_model_pose>true</publish_model_pose>
@@ -44,5 +51,5 @@
     </plugin>
   </gazebo>
-  <!-- Definindo a Base do Robô -->
+  <!-- Definindo a base do robô -->
   <link name="base_link">
     <visual>
@@ -61,5 +68,5 @@
     <xacro:box_inertia m="1" w="${base_width}" d="${base_length}" h="${base_height}"/>
   </link>
-  <!-- Definindo a Base do Robô (base footprint) -->
+  <!-- Definição da base footprint -->
   <link name="base_footprint">
     <xacro:box_inertia m="0" w="0" d="0" h="0"/>
@@ -68,8 +75,7 @@
     <parent link="base_link"/>
     <child link="base_footprint"/>
-    <origin xyz="0.0 0.0 ${-(wheel_radius+wheel_zoff)}" rpy="0 0 0"/>
-  </joint>
-  <!-- Definindo as Rodas do Robô -->
-  <!-- Parâmetros: prefix: drivewhl_l, drivewhl_r -->
+    <origin xyz="0.0 0.0 ${-(wheel_radius + wheel_zoff)}" rpy="0 0 0"/>
+  </joint>
+  <!-- Definindo as rodas do robô -->
   <xacro:macro name="wheel" params="prefix x_reflect y_reflect">
     <link name="${prefix}_link">
@@ -94,15 +100,21 @@
       <parent link="base_link"/>
       <child link="${prefix}_link"/>
-      <origin xyz="${x_reflect*wheel_xoff} ${y_reflect*(base_width/2+wheel_ygap)} ${-wheel_zoff}" rpy="0 0 0"/>
+      <origin xyz="${x_reflect * wheel_xoff}
+                    ${y_reflect * (base_width/2 + wheel_ygap)}
+                    ${-wheel_zoff}"
+              rpy="0 0 0"/>
       <axis xyz="0 1 0"/>
       <dynamics damping="0.2"/>
     </joint>
   </xacro:macro>
+  <!-- Rodas esquerda e direita -->
   <xacro:wheel prefix="drivewhl_l" x_reflect="-1" y_reflect="1" />
   <xacro:wheel prefix="drivewhl_r" x_reflect="-1" y_reflect="-1" />
+  <!-- Definindo o caster frontu -->
   <link name="front_caster">
     <visual>
       <geometry>
-        <sphere radius="${(wheel_radius+wheel_zoff-(base_height/2))}"/>
+        <!-- O raio do caster permanece calculado como antes -->
+        <sphere radius="${(wheel_radius + wheel_zoff - (base_height/2))}"/>
       </geometry>
       <material name="DarkBlue">
@@ -113,8 +125,8 @@
       <origin xyz="0 0 0" rpy="0 0 0"/>
       <geometry>
-        <sphere radius="${(wheel_radius+wheel_zoff-(base_height/2))}"/>
-      </geometry>
-    </collision>
-    <xacro:sphere_inertia m="0.005" r="${(wheel_radius+wheel_zoff-(base_height/2))}"/>
+        <sphere radius="${(wheel_radius + wheel_zoff - (base_height/2))}"/>
+      </geometry>
+    </collision>
+    <xacro:sphere_inertia m="0.005" r="${(wheel_radius + wheel_zoff - (base_height/2))}"/>
   </link>
   <joint name="caster_joint" type="fixed">
@@ -123,5 +135,5 @@
     <origin xyz="${caster_xoff} 0.0 ${-(base_height/2)}" rpy="0 0 0"/>
   </joint>
-  <!-- Definindo a IMU do Robô (física) -->
+  <!-- Definindo a IMU do robô -->
   <link name="imu_link">
     <visual>
@@ -137,10 +149,10 @@
     <xacro:box_inertia m="0.001" w="0.1" d="0.1" h="0.1"/>
   </link>
-  <!-- Definindo o sensor IMU no Gazebo -->
+  <!-- Sensor IMU no Gazebo/Ignition -->
   <gazebo reference="imu_link">
     <sensor name="imu_sensor" type="imu">
       <ignition_frame_id>imu_link</ignition_frame_id>
-      <plugin filename="ignition-gazebo-imu-system" name="ignition::gazebo::systems::Imu">
-      </plugin>
+      <plugin filename="ignition-gazebo-imu-system"
+              name="ignition::gazebo::systems::Imu"/>
       <topic>imu</topic>
       <always_on>true</always_on>
@@ -203,56 +215,44 @@
     </sensor>
   </gazebo>
-  <!-- Ligando a IMU a base do robô -->
+  <!-- Ligando a IMU à base do robô -->
   <joint name="imu_joint" type="fixed">
     <parent link="base_link"/>
     <child link="imu_link"/>
-    <origin xyz="0 0 0.01"/>
-  </joint>
-<!-- Define um sistema de controle ROS 2 utilizando a infraestrutura ros2_control -->
-<ros2_control name="IgnitionSystem" type="system">
-  <!-- Seção de hardware do sistema, onde é especificado o plugin que fará a ponte entre o Gazebo (Ignition) e o ros2_control -->
-  <hardware>
-    <!-- Plugin que permite a integração entre o Ignition Gazebo e o framework ros2_control -->
-    <plugin>ign_ros2_control/IgnitionSystem</plugin>
-  </hardware>
-  <!-- Definição do primeiro atuador, correspondente à roda esquerda ("drive wheel left") -->
-  <joint name="drivewhl_l_joint">
-    <!-- Interface de comando de velocidade angular (por exemplo, rad/s) para essa junta -->
-    <command_interface name="velocity">
-      <!-- Valor mínimo permitido para o comando de velocidade (limite inferior) -->
-      <param name="min">-1</param>
-      <!-- Valor máximo permitido para o comando de velocidade (limite superior) -->
-      <param name="max">1</param>
-    </command_interface>
-    <!-- Interface de estado que fornece a posição atual da junta (por exemplo, em radianos) -->
-    <state_interface name="position"/>
-    <!-- Interface de estado que fornece a velocidade atual da junta (por exemplo, em rad/s) -->
-    <state_interface name="velocity"/>
-  </joint>
-  <!-- Definição do segundo atuador, correspondente à roda direita ("drive wheel right") -->
-  <joint name="drivewhl_r_joint">
-    <!-- Interface de comando de velocidade angular para essa junta -->
-    <command_interface name="velocity">
-      <!-- Limite inferior da velocidade que pode ser comandada -->
-      <param name="min">-1</param>
-      <!-- Limite superior da velocidade que pode ser comandada -->
-      <param name="max">1</param>
-    </command_interface>
-    <!-- Interface de estado para leitura da posição da junta -->
-    <state_interface name="position"/>
-    <!-- Interface de estado para leitura da velocidade da junta -->
-    <state_interface name="velocity"/>
-  </joint>
-</ros2_control>
+    <origin xyz="0 0 0.01" rpy="0 0 0"/>
+  </joint>
+  <!-- Sistemas ros2_control (ros2_control + Ignition) -->
+  <ros2_control name="IgnitionSystem" type="system">
+    <hardware>
+      <plugin>ign_ros2_control/IgnitionSystem</plugin>
+    </hardware>
+    <joint name="drivewhl_l_joint">
+      <command_interface name="velocity">
+        <param name="min">-1</param>
+        <param name="max">1</param>
+      </command_interface>
+      <state_interface name="position"/>
+      <state_interface name="velocity"/>
+    </joint>
+    <joint name="drivewhl_r_joint">
+      <command_interface name="velocity">
+        <param name="min">-1</param>
+        <param name="max">1</param>
+      </command_interface>
+      <state_interface name="position"/>
+      <state_interface name="velocity"/>
+    </joint>
+  </ros2_control>
   <gazebo>
-    <plugin filename="ign_ros2_control-system" name="ign_ros2_control::IgnitionROS2ControlPlugin">
+    <plugin filename="ign_ros2_control-system"
+            name="ign_ros2_control::IgnitionROS2ControlPlugin">
       <parameters>$(find prm)/config/diff_drive_controller_velocity.yaml</parameters>
     </plugin>
   </gazebo>
+  <!-- Definindo o LIDAR -->
   <link name="lidar_link">
     <inertial>
       <origin xyz="0 0 0" rpy="0 0 0"/>
       <mass value="0.125"/>
-      <inertia ixx="0.001" ixy="0" ixz="0" iyy="0.001" iyz="0" izz="0.001" />
+      <inertia ixx="0.001" ixy="0" ixz="0" iyy="0.001" iyz="0" izz="0.001"/>
     </inertial>
     <collision>
@@ -306,4 +306,5 @@
     </sensor>
   </gazebo>
+  <!-- Definindo a câmera frontal -->
   <link name="camera_link">
     <visual>
@@ -325,5 +326,5 @@
       <origin xyz="0 0 0" rpy="0 0 0"/>
       <mass value="0.035"/>
-      <inertia ixx="0.001" ixy="0" ixz="0" iyy="0.001" iyz="0" izz="0.001" />
+      <inertia ixx="0.001" ixy="0" ixz="0" iyy="0.001" iyz="0" izz="0.001"/>
     </inertial>
   </link>
@@ -331,5 +332,6 @@
     <parent link="base_link"/>
     <child link="camera_link"/>
-    <origin xyz="0.215 0 0.05" rpy="0 0 0"/>
+    <!-- Ajustada a posição X da câmera para metade do comprimento da base -->
+    <origin xyz="0.105 0 0.05" rpy="0 0 0"/>
   </joint>
   <link name="camera_frame"/>
@@ -340,24 +342,5 @@
   </joint>
   <gazebo reference="camera_link">
-    <!-- Insere uma camera comum RGB -->
-    <!-- <sensor name="robot_cam" type="camera">
-      <camera>
-        <horizontal_fov>1.57</horizontal_fov>
-        <image>
-          <width>320</width>
-          <height>240</height>
-        </image>
-        <clip>
-          <near>0.1</near>
-          <far>100</far>
-        </clip>
-      </camera>
-      <always_on>1</always_on>
-      <update_rate>15</update_rate>
-      <visualize>true</visualize>
-      <topic>robot_cam</topic>
-      <enable_metrics>true</enable_metrics>
-    </sensor> -->
-    <!-- Insere uma camera com segmentacao semantica -->
+    <!-- Câmera com segmentação semântica -->
     <sensor name="robot_cam" type="segmentation">
       <topic>robot_cam</topic>
@@ -378,70 +361,4 @@
       <visualize>true</visualize>
     </sensor>
-    <!-- Insere uma camera bounding box 2D completo -->
-    <!-- <sensor name="full_2d" type="boundingbox_camera">
-      <topic>boxes_full_2d</topic>
-      <camera>
-        <box_type>full_2d</box_type>
-        <horizontal_fov>1.57</horizontal_fov>
-        <image>
-          <width>320</width>
-          <height>240</height>
-        </image>
-        <clip>
-          <near>0.1</near>
-          <far>10</far>
-        </clip>
-        <save enabled="false">
-          <path>bounding_box_full_2d_data</path>
-        </save>
-      </camera>
-      <always_on>1</always_on>
-      <update_rate>15</update_rate>
-      <visualize>true</visualize>
-    </sensor> -->
-    <!-- Insere uma camera bounding box 2D -->
-    <!-- <sensor name="visible_2d" type="boundingbox_camera">
-      <topic>boxes_visible_2d</topic>
-      <camera>
-        <box_type>visible_2d</box_type>
-        <horizontal_fov>1.57</horizontal_fov>
-        <image>
-          <width>320</width>
-          <height>240</height>
-        </image>
-        <clip>
-          <near>0.1</near>
-          <far>10</far>
-        </clip>
-        <save enabled="false">
-          <path>bounding_box_visible_2d_data</path>
-        </save>
-      </camera>
-      <always_on>1</always_on>
-      <update_rate>15</update_rate>
-      <visualize>true</visualize>
-    </sensor> -->
-    <!-- Insere uma camera bounding box 3D -->
-    <!-- <sensor name="3d" type="boundingbox_camera">
-      <topic>boxes_3d</topic>
-      <camera>
-        <box_type>3d</box_type>
-        <horizontal_fov>1.57</horizontal_fov>
-        <image>
-          <width>320</width>
-          <height>240</height>
-        </image>
-        <clip>
-          <near>0.1</near>
-          <far>10</far>
-        </clip>
-        <save enabled="false">
-          <path>bounding_box_3d_data</path>
-        </save>
-      </camera>
-      <always_on>1</always_on>
-      <update_rate>15</update_rate>
-      <visualize>true</visualize>
-    </sensor> -->
   </gazebo>
 </robot>

Commit message: primeiro commit da versao final

File: description/robot.urdf.xacro (robot description, xacro)
@@ -3,6 +3,6 @@
   xmlns:xacro="http://ros.org/wiki/xacro">
   <!-- Definicao de Algumas Contantes -->
-  <xacro:property name="base_width" value="0.21"/> <!-- Largura da base -->
-  <xacro:property name="base_length" value="0.42"/> <!-- Comprimento da base -->
+  <xacro:property name="base_width" value="0.11"/> <!-- Largura da base -->
+  <xacro:property name="base_length" value="0.32"/> <!-- Comprimento da base -->
   <xacro:property name="base_height" value="0.18"/> <!-- Altura da base -->
   <xacro:property name="wheel_radius" value="0.10"/> <!-- Raio da roda -->
