Commit message: iniciando t2

File: description/robot.urdf.xacro (robot description, xacro)
@@ -2,14 +2,14 @@
 <robot name="prm_robot"
   xmlns:xacro="http://ros.org/wiki/xacro">
-  <!-- Definição de algumas constantes (comprimento e largura reduzidos pela metade, altura mantida) -->
-  <xacro:property name="base_width" value="0.155"/> <!-- Largura da base (original 0.31 reduzido para 0.155) -->
-  <xacro:property name="base_length" value="0.21"/> <!-- Comprimento da base (original 0.42 reduzido para 0.21) -->
-  <xacro:property name="base_height" value="0.18"/> <!-- Altura da base (permanece 0.18) -->
-  <xacro:property name="wheel_radius" value="0.10"/> <!-- Raio da roda (permanece 0.10) -->
-  <xacro:property name="wheel_width" value="0.04"/>  <!-- Largura da roda (permanece 0.04) -->
-  <xacro:property name="wheel_ygap" value="0.0125"/> <!-- Distância entre as rodas em Y (original 0.025 reduzido para 0.0125) -->
-  <xacro:property name="wheel_zoff" value="0.05"/>   <!-- Deslocamento da roda em Z (permanece 0.05) -->
-  <xacro:property name="wheel_xoff" value="0.06"/>   <!-- Deslocamento da roda em X (original 0.12 reduzido para 0.06) -->
-  <xacro:property name="caster_xoff" value="0.07"/> <!-- Deslocamento do caster em X (original 0.14 reduzido para 0.07) -->
+  <!-- Definicao de Algumas Contantes -->
+  <xacro:property name="base_width" value="0.11"/> <!-- Largura da base -->
+  <xacro:property name="base_length" value="0.42"/> <!-- Comprimento da base -->
+  <xacro:property name="base_height" value="0.18"/> <!-- Altura da base -->
+  <xacro:property name="wheel_radius" value="0.10"/> <!-- Raio da roda -->
+  <xacro:property name="wheel_width" value="0.04"/> <!-- Largura da roda -->
+  <xacro:property name="wheel_ygap" value="0.025"/> <!-- Distancia entre as rodas -->
+  <xacro:property name="wheel_zoff" value="0.05"/> <!-- Deslocamento da roda em Z -->
+  <xacro:property name="wheel_xoff" value="0.12"/> <!-- Deslocamento da roda em X -->
+  <xacro:property name="caster_xoff" value="0.14"/> <!-- Deslocamento do caster em X -->
   <!-- Definição de algumas propriedades inerciais -->
   <xacro:macro name="box_inertia" params="m w h d">
@@ -17,16 +17,12 @@
       <origin xyz="0 0 0" rpy="${pi/2} 0 ${pi/2}"/>
       <mass value="${m}"/>
-      <inertia ixx="${(m/12) * (h*h + d*d)}" ixy="0.0" ixz="0.0"
-               iyy="${(m/12) * (w*w + d*d)}" iyz="0.0"
-               izz="${(m/12) * (w*w + h*h)}"/>
+      <inertia ixx="${(m/12) * (h*h + d*d)}" ixy="0.0" ixz="0.0" iyy="${(m/12) * (w*w + d*d)}" iyz="0.0" izz="${(m/12) * (w*w + h*h)}"/>
     </inertial>
   </xacro:macro>
   <xacro:macro name="cylinder_inertia" params="m r h">
     <inertial>
-      <origin xyz="0 0 0" rpy="${pi/2} 0 0"/>
+      <origin xyz="0 0 0" rpy="${pi/2} 0 0" />
       <mass value="${m}"/>
-      <inertia ixx="${(m/12) * (3*r*r + h*h)}" ixy="0" ixz="0"
-               iyy="${(m/12) * (3*r*r + h*h)}" iyz="0"
-               izz="${(m/2) * (r*r)}"/>
+      <inertia ixx="${(m/12) * (3*r*r + h*h)}" ixy = "0" ixz = "0" iyy="${(m/12) * (3*r*r + h*h)}" iyz = "0" izz="${(m/2) * (r*r)}"/>
     </inertial>
   </xacro:macro>
@@ -34,13 +30,10 @@
     <inertial>
       <mass value="${m}"/>
-      <inertia ixx="${(2/5) * m * (r*r)}" ixy="0.0" ixz="0.0"
-               iyy="${(2/5) * m * (r*r)}" iyz="0.0"
-               izz="${(2/5) * m * (r*r)}"/>
+      <inertia ixx="${(2/5) * m * (r*r)}" ixy="0.0" ixz="0.0" iyy="${(2/5) * m * (r*r)}" iyz="0.0" izz="${(2/5) * m * (r*r)}"/>
     </inertial>
   </xacro:macro>
-  <!-- Plugin do Gazebo/Ignition para publicar pose do robô -->
+  <!-- Definindo plugin para publiar a pose do robo -->
   <gazebo>
-    <plugin filename="libignition-gazebo-pose-publisher-system"
-            name="ignition::gazebo::systems::PosePublisher">
+    <plugin filename="libignition-gazebo-pose-publisher-system" name="ignition::gazebo::systems::PosePublisher">
       <publish_link_pose>false</publish_link_pose>
       <publish_model_pose>true</publish_model_pose>
@@ -51,5 +44,5 @@
     </plugin>
   </gazebo>
-  <!-- Definindo a base do robô -->
+  <!-- Definindo a Base do Robô -->
   <link name="base_link">
     <visual>
@@ -68,5 +61,5 @@
     <xacro:box_inertia m="1" w="${base_width}" d="${base_length}" h="${base_height}"/>
   </link>
-  <!-- Definição da base footprint -->
+  <!-- Definindo a Base do Robô (base footprint) -->
   <link name="base_footprint">
     <xacro:box_inertia m="0" w="0" d="0" h="0"/>
@@ -75,7 +68,8 @@
     <parent link="base_link"/>
     <child link="base_footprint"/>
-    <origin xyz="0.0 0.0 ${-(wheel_radius + wheel_zoff)}" rpy="0 0 0"/>
-  </joint>
-  <!-- Definindo as rodas do robô -->
+    <origin xyz="0.0 0.0 ${-(wheel_radius+wheel_zoff)}" rpy="0 0 0"/>
+  </joint>
+  <!-- Definindo as Rodas do Robô -->
+  <!-- Parâmetros: prefix: drivewhl_l, drivewhl_r -->
   <xacro:macro name="wheel" params="prefix x_reflect y_reflect">
     <link name="${prefix}_link">
@@ -100,21 +94,15 @@
       <parent link="base_link"/>
       <child link="${prefix}_link"/>
-      <origin xyz="${x_reflect * wheel_xoff}
-                    ${y_reflect * (base_width/2 + wheel_ygap)}
-                    ${-wheel_zoff}"
-              rpy="0 0 0"/>
+      <origin xyz="${x_reflect*wheel_xoff} ${y_reflect*(base_width/2+wheel_ygap)} ${-wheel_zoff}" rpy="0 0 0"/>
       <axis xyz="0 1 0"/>
       <dynamics damping="0.2"/>
     </joint>
   </xacro:macro>
-  <!-- Rodas esquerda e direita -->
   <xacro:wheel prefix="drivewhl_l" x_reflect="-1" y_reflect="1" />
   <xacro:wheel prefix="drivewhl_r" x_reflect="-1" y_reflect="-1" />
-  <!-- Definindo o caster frontu -->
   <link name="front_caster">
     <visual>
       <geometry>
-        <!-- O raio do caster permanece calculado como antes -->
-        <sphere radius="${(wheel_radius + wheel_zoff - (base_height/2))}"/>
+        <sphere radius="${(wheel_radius+wheel_zoff-(base_height/2))}"/>
       </geometry>
       <material name="DarkBlue">
@@ -125,8 +113,8 @@
       <origin xyz="0 0 0" rpy="0 0 0"/>
       <geometry>
-        <sphere radius="${(wheel_radius + wheel_zoff - (base_height/2))}"/>
-      </geometry>
-    </collision>
-    <xacro:sphere_inertia m="0.005" r="${(wheel_radius + wheel_zoff - (base_height/2))}"/>
+        <sphere radius="${(wheel_radius+wheel_zoff-(base_height/2))}"/>
+      </geometry>
+    </collision>
+    <xacro:sphere_inertia m="0.005" r="${(wheel_radius+wheel_zoff-(base_height/2))}"/>
   </link>
   <joint name="caster_joint" type="fixed">
@@ -135,5 +123,5 @@
     <origin xyz="${caster_xoff} 0.0 ${-(base_height/2)}" rpy="0 0 0"/>
   </joint>
-  <!-- Definindo a IMU do robô -->
+  <!-- Definindo a IMU do Robô (física) -->
   <link name="imu_link">
     <visual>
@@ -149,10 +137,10 @@
     <xacro:box_inertia m="0.001" w="0.1" d="0.1" h="0.1"/>
   </link>
-  <!-- Sensor IMU no Gazebo/Ignition -->
+  <!-- Definindo o sensor IMU no Gazebo -->
   <gazebo reference="imu_link">
     <sensor name="imu_sensor" type="imu">
       <ignition_frame_id>imu_link</ignition_frame_id>
-      <plugin filename="ignition-gazebo-imu-system"
-              name="ignition::gazebo::systems::Imu"/>
+      <plugin filename="ignition-gazebo-imu-system" name="ignition::gazebo::systems::Imu">
+      </plugin>
       <topic>imu</topic>
       <always_on>true</always_on>
@@ -215,27 +203,65 @@
     </sensor>
   </gazebo>
-  <!-- Ligando a IMU à base do robô -->
+  <!-- Ligando a IMU a base do robô -->
   <joint name="imu_joint" type="fixed">
     <parent link="base_link"/>
     <child link="imu_link"/>
-    <origin xyz="0 0 0.01" rpy="0 0 0"/>
-  </joint>
-  <!-- Sistemas ros2_control (ros2_control + Ignition) -->
+    <origin xyz="0 0 0.01"/>
+  </joint>
+  <!-- Define um sistema de controle ROS 2 utilizando a infraestrutura ros2_control -->
   <ros2_control name="IgnitionSystem" type="system">
+    <!-- Seção de hardware do sistema, onde é especificado o plugin que fará a ponte entre o Gazebo (Ignition) e o ros2_control -->
     <hardware>
+      <!-- Plugin que permite a integração entre o Ignition Gazebo e o framework ros2_control -->
       <plugin>ign_ros2_control/IgnitionSystem</plugin>
     </hardware>
+    <!-- Definição do primeiro atuador, correspondente à roda esquerda ("drive wheel left") -->
     <joint name="drivewhl_l_joint">
+      <!-- Interface de comando de velocidade angular (por exemplo, rad/s) para essa junta -->
       <command_interface name="velocity">
+        <!-- Valor mínimo permitido para o comando de velocidade (limite inferior) -->
         <param name="min">-1</param>
+        <!-- Valor máximo permitido para o comando de velocidade (limite superior) -->
         <param name="max">1</param>
+      </command_interface>
+      <!-- Interface de estado que fornece a posição atual da junta (por exemplo, em radianos) -->
+      <state_interface name="position"/>
+      <!-- Interface de estado que fornece a velocidade atual da junta (por exemplo, em rad/s) -->
+      <state_interface name="velocity"/>
+    </joint>
+    <!-- Definição do segundo atuador, correspondente à roda direita ("drive wheel right") -->
+    <joint name="drivewhl_r_joint">
+      <!-- Interface de comando de velocidade angular para essa junta -->
+      <command_interface name="velocity">
+        <!-- Limite inferior da velocidade que pode ser comandada -->
+        <param name="min">-1</param>
+        <!-- Limite superior da velocidade que pode ser comandada -->
+        <param name="max">1</param>
+      </command_interface>
+      <!-- Interface de estado para leitura da posição da junta -->
+      <state_interface name="position"/>
+      <!-- Interface de estado para leitura da velocidade da junta -->
+      <state_interface name="velocity"/>
+    </joint>
+    <joint name="gripper_extension">
+      <command_interface name="position">
+        <param name="min">-1.57075</param>
+        <param name="max">0.2</param>
       </command_interface>
       <state_interface name="position"/>
       <state_interface name="velocity"/>
     </joint>
-    <joint name="drivewhl_r_joint">
-      <command_interface name="velocity">
-        <param name="min">-1</param>
-        <param name="max">1</param>
+    <joint name="left_gripper_joint">
+      <command_interface name="position">
+        <param name="min">0.0</param>
+        <param name="max">0.06</param>
+      </command_interface>
+      <state_interface name="position"/>
+      <state_interface name="velocity"/>
+    </joint>
+    <joint name="right_gripper_joint">
+      <command_interface name="position">
+        <param name="min">-0.06</param>
+        <param name="max">0.0</param>
       </command_interface>
       <state_interface name="position"/>
@@ -244,15 +270,13 @@
   </ros2_control>
   <gazebo>
-    <plugin filename="ign_ros2_control-system"
-            name="ign_ros2_control::IgnitionROS2ControlPlugin">
+    <plugin filename="ign_ros2_control-system" name="ign_ros2_control::IgnitionROS2ControlPlugin">
       <parameters>$(find prm)/config/diff_drive_controller_velocity.yaml</parameters>
     </plugin>
   </gazebo>
-  <!-- Definindo o LIDAR -->
   <link name="lidar_link">
     <inertial>
       <origin xyz="0 0 0" rpy="0 0 0"/>
       <mass value="0.125"/>
-      <inertia ixx="0.001" ixy="0" ixz="0" iyy="0.001" iyz="0" izz="0.001"/>
+      <inertia ixx="0.001" ixy="0" ixz="0" iyy="0.001" iyz="0" izz="0.001" />
     </inertial>
     <collision>
@@ -306,5 +330,4 @@
     </sensor>
   </gazebo>
-  <!-- Definindo a câmera frontal -->
   <link name="camera_link">
     <visual>
@@ -326,5 +349,5 @@
       <origin xyz="0 0 0" rpy="0 0 0"/>
       <mass value="0.035"/>
-      <inertia ixx="0.001" ixy="0" ixz="0" iyy="0.001" iyz="0" izz="0.001"/>
+      <inertia ixx="0.001" ixy="0" ixz="0" iyy="0.001" iyz="0" izz="0.001" />
     </inertial>
   </link>
@@ -332,6 +355,5 @@
     <parent link="base_link"/>
     <child link="camera_link"/>
-    <!-- Ajustada a posição X da câmera para metade do comprimento da base -->
-    <origin xyz="0.105 0 0.05" rpy="0 0 0"/>
+    <origin xyz="0.215 0 0.05" rpy="0 0 0"/>
   </joint>
   <link name="camera_frame"/>
@@ -342,5 +364,24 @@
   </joint>
   <gazebo reference="camera_link">
-    <!-- Câmera com segmentação semântica -->
+    <!-- Insere uma camera comum RGB -->
+    <!-- <sensor name="robot_cam" type="camera">
+      <camera>
+        <horizontal_fov>1.57</horizontal_fov>
+        <image>
+          <width>320</width>
+          <height>240</height>
+        </image>
+        <clip>
+          <near>0.1</near>
+          <far>100</far>
+        </clip>
+      </camera>
+      <always_on>1</always_on>
+      <update_rate>15</update_rate>
+      <visualize>true</visualize>
+      <topic>robot_cam</topic>
+      <enable_metrics>true</enable_metrics>
+    </sensor> -->
+    <!-- Insere uma camera com segmentacao semantica -->
     <sensor name="robot_cam" type="segmentation">
       <topic>robot_cam</topic>
@@ -361,4 +402,173 @@
       <visualize>true</visualize>
     </sensor>
+    <!-- Insere uma camera bounding box 2D completo -->
+    <!-- <sensor name="full_2d" type="boundingbox_camera">
+      <topic>boxes_full_2d</topic>
+      <camera>
+        <box_type>full_2d</box_type>
+        <horizontal_fov>1.57</horizontal_fov>
+        <image>
+          <width>320</width>
+          <height>240</height>
+        </image>
+        <clip>
+          <near>0.1</near>
+          <far>10</far>
+        </clip>
+        <save enabled="false">
+          <path>bounding_box_full_2d_data</path>
+        </save>
+      </camera>
+      <always_on>1</always_on>
+      <update_rate>15</update_rate>
+      <visualize>true</visualize>
+    </sensor> -->
+    <!-- Insere uma camera bounding box 2D -->
+    <!-- <sensor name="visible_2d" type="boundingbox_camera">
+      <topic>boxes_visible_2d</topic>
+      <camera>
+        <box_type>visible_2d</box_type>
+        <horizontal_fov>1.57</horizontal_fov>
+        <image>
+          <width>320</width>
+          <height>240</height>
+        </image>
+        <clip>
+          <near>0.1</near>
+          <far>10</far>
+        </clip>
+        <save enabled="false">
+          <path>bounding_box_visible_2d_data</path>
+        </save>
+      </camera>
+      <always_on>1</always_on>
+      <update_rate>15</update_rate>
+      <visualize>true</visualize>
+    </sensor> -->
+    <!-- Insere uma camera bounding box 3D -->
+    <!-- <sensor name="3d" type="boundingbox_camera">
+      <topic>boxes_3d</topic>
+      <camera>
+        <box_type>3d</box_type>
+        <horizontal_fov>1.57</horizontal_fov>
+        <image>
+          <width>320</width>
+          <height>240</height>
+        </image>
+        <clip>
+          <near>0.1</near>
+          <far>10</far>
+        </clip>
+        <save enabled="false">
+          <path>bounding_box_3d_data</path>
+        </save>
+      </camera>
+      <always_on>1</always_on>
+      <update_rate>15</update_rate>
+      <visualize>true</visualize>
+    </sensor> -->
   </gazebo>
+  <joint name="gripper_extension" type="revolute">
+    <axis xyz="0 1 0"/>
+    <limit effort="50.0" lower="-1.57075" upper="0.2" velocity="0.5"/>
+    <origin rpy="0 0 0" xyz="0.2 0 0.1"/>
+    <parent link="base_link"/>
+    <child link="gripper_pole"/>
+  </joint>
+  <link name="gripper_pole">
+    <visual>
+      <geometry>
+        <cylinder length="0.2" radius="0.01"/>
+      </geometry>
+      <origin rpy="0 1.57075 0" xyz="0.1 0 0"/>
+    </visual>
+    <collision>
+      <geometry>
+        <cylinder length="0.2" radius="0.01"/>
+      </geometry>
+    </collision>
+    <xacro:cylinder_inertia m="0.01" r="0.01" h="0.2"/>
+  </link>
+  <joint name="left_gripper_joint" type="prismatic">
+    <axis xyz="0 1 0"/>
+    <limit effort="100.0" lower="0.0" upper="0.06" velocity="0.25"/>
+    <origin rpy="0 0 0" xyz="0.2 0.01 0"/>
+    <parent link="gripper_pole"/>
+    <child link="left_gripper"/>
+  </joint>
+  <link name="left_gripper">
+    <visual>
+      <geometry>
+        <box size="0.1 0.02 0.02"/> <!-- Comprimento, largura, altura -->
+      </geometry>
+    </visual>
+    <collision>
+      <geometry>
+        <box size="0.1 0.02 0.02"/>
+      </geometry>
+    </collision>
+    <xacro:box_inertia m="0.015" w="0.02" h="0.02" d="0.1"/>
+  </link>
+  <joint name="left_tip_joint" type="fixed">
+    <origin rpy="0.0 0 0" xyz="0.06 0.001 0"/>
+    <parent link="left_gripper"/>
+    <child link="left_tip"/>
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
Commit message: arrumando área de colisao do gripper

File: description/robot.urdf.xacro (robot description, xacro)
@@ -484,4 +484,5 @@
     </visual>
     <collision>
+      <origin rpy="0 1.57075 0" xyz="0.1 0 0"/>
       <geometry>
         <cylinder length="0.2" radius="0.01"/>

Commit message: versao funcional arena tartaruga

File: description/robot.urdf.xacro (robot description, xacro)
@@ -4,5 +4,5 @@
   <!-- Definicao de Algumas Contantes -->
   <xacro:property name="base_width" value="0.11"/> <!-- Largura da base -->
-  <xacro:property name="base_length" value="0.42"/> <!-- Comprimento da base -->
+  <xacro:property name="base_length" value="0.12"/> <!-- Comprimento da base -->
   <xacro:property name="base_height" value="0.18"/> <!-- Altura da base -->
   <xacro:property name="wheel_radius" value="0.10"/> <!-- Raio da roda -->
@@ -472,5 +472,5 @@
     <axis xyz="0 1 0"/>
     <limit effort="50.0" lower="-1.57075" upper="0.2" velocity="0.5"/>
-    <origin rpy="0 0 0" xyz="0.2 0 0.1"/>
+    <origin rpy="0 0 0" xyz="0.05 0 0.1"/>
     <parent link="base_link"/>
     <child link="gripper_pole"/>
@@ -479,5 +479,5 @@
     <visual>
       <geometry>
-        <cylinder length="0.2" radius="0.01"/>
+        <cylinder length="0.1" radius="0.01"/>
       </geometry>
       <origin rpy="0 1.57075 0" xyz="0.1 0 0"/>
