Commit message: merging_into_main

File: description/robot.urdf.xacro (robot description, xacro)
@@ -4,5 +4,5 @@
   <!-- Definicao de Algumas Contantes -->
   <xacro:property name="base_width" value="0.11"/> <!-- Largura da base -->
-  <xacro:property name="base_length" value="0.32"/> <!-- Comprimento da base -->
+  <xacro:property name="base_length" value="0.12"/> <!-- Comprimento da base -->
   <xacro:property name="base_height" value="0.18"/> <!-- Altura da base -->
   <xacro:property name="wheel_radius" value="0.10"/> <!-- Raio da roda -->
@@ -209,40 +209,64 @@
     <origin xyz="0 0 0.01"/>
   </joint>
-<!-- Define um sistema de controle ROS 2 utilizando a infraestrutura ros2_control -->
-<ros2_control name="IgnitionSystem" type="system">
-  <!-- Seção de hardware do sistema, onde é especificado o plugin que fará a ponte entre o Gazebo (Ignition) e o ros2_control -->
-  <hardware>
-    <!-- Plugin que permite a integração entre o Ignition Gazebo e o framework ros2_control -->
-    <plugin>ign_ros2_control/IgnitionSystem</plugin>
-  </hardware>
-  <!-- Definição do primeiro atuador, correspondente à roda esquerda ("drive wheel left") -->
-  <joint name="drivewhl_l_joint">
-    <!-- Interface de comando de velocidade angular (por exemplo, rad/s) para essa junta -->
-    <command_interface name="velocity">
-      <!-- Valor mínimo permitido para o comando de velocidade (limite inferior) -->
-      <param name="min">-1</param>
-      <!-- Valor máximo permitido para o comando de velocidade (limite superior) -->
-      <param name="max">1</param>
-    </command_interface>
-    <!-- Interface de estado que fornece a posição atual da junta (por exemplo, em radianos) -->
-    <state_interface name="position"/>
-    <!-- Interface de estado que fornece a velocidade atual da junta (por exemplo, em rad/s) -->
-    <state_interface name="velocity"/>
-  </joint>
-  <!-- Definição do segundo atuador, correspondente à roda direita ("drive wheel right") -->
-  <joint name="drivewhl_r_joint">
-    <!-- Interface de comando de velocidade angular para essa junta -->
-    <command_interface name="velocity">
-      <!-- Limite inferior da velocidade que pode ser comandada -->
-      <param name="min">-1</param>
-      <!-- Limite superior da velocidade que pode ser comandada -->
-      <param name="max">1</param>
-    </command_interface>
-    <!-- Interface de estado para leitura da posição da junta -->
-    <state_interface name="position"/>
-    <!-- Interface de estado para leitura da velocidade da junta -->
-    <state_interface name="velocity"/>
-  </joint>
-</ros2_control>
+  <!-- Define um sistema de controle ROS 2 utilizando a infraestrutura ros2_control -->
+  <ros2_control name="IgnitionSystem" type="system">
+    <!-- Seção de hardware do sistema, onde é especificado o plugin que fará a ponte entre o Gazebo (Ignition) e o ros2_control -->
+    <hardware>
+      <!-- Plugin que permite a integração entre o Ignition Gazebo e o framework ros2_control -->
+      <plugin>ign_ros2_control/IgnitionSystem</plugin>
+    </hardware>
+    <!-- Definição do primeiro atuador, correspondente à roda esquerda ("drive wheel left") -->
+    <joint name="drivewhl_l_joint">
+      <!-- Interface de comando de velocidade angular (por exemplo, rad/s) para essa junta -->
+      <command_interface name="velocity">
+        <!-- Valor mínimo permitido para o comando de velocidade (limite inferior) -->
+        <param name="min">-1</param>
+        <!-- Valor máximo permitido para o comando de velocidade (limite superior) -->
+        <param name="max">1</param>
+      </command_interface>
+      <!-- Interface de estado que fornece a posição atual da junta (por exemplo, em radianos) -->
+      <state_interface name="position"/>
+      <!-- Interface de estado que fornece a velocidade atual da junta (por exemplo, em rad/s) -->
+      <state_interface name="velocity"/>
+    </joint>
+    <!-- Definição do segundo atuador, correspondente à roda direita ("drive wheel right") -->
+    <joint name="drivewhl_r_joint">
+      <!-- Interface de comando de velocidade angular para essa junta -->
+      <command_interface name="velocity">
+        <!-- Limite inferior da velocidade que pode ser comandada -->
+        <param name="min">-1</param>
+        <!-- Limite superior da velocidade que pode ser comandada -->
+        <param name="max">1</param>
+      </command_interface>
+      <!-- Interface de estado para leitura da posição da junta -->
+      <state_interface name="position"/>
+      <!-- Interface de estado para leitura da velocidade da junta -->
+      <state_interface name="velocity"/>
+    </joint>
+    <joint name="gripper_extension">
+      <command_interface name="position">
+        <param name="min">-1.57075</param>
+        <param name="max">0.2</param>
+      </command_interface>
+      <state_interface name="position"/>
+      <state_interface name="velocity"/>
+    </joint>
+    <joint name="left_gripper_joint">
+      <command_interface name="position">
+        <param name="min">0.0</param>
+        <param name="max">0.06</param>
+      </command_interface>
+      <state_interface name="position"/>
+      <state_interface name="velocity"/>
+    </joint>
+    <joint name="right_gripper_joint">
+      <command_interface name="position">
+        <param name="min">-0.06</param>
+        <param name="max">0.0</param>
+      </command_interface>
+      <state_interface name="position"/>
+      <state_interface name="velocity"/>
+    </joint>
+  </ros2_control>
   <gazebo>
     <plugin filename="ign_ros2_control-system" name="ign_ros2_control::IgnitionROS2ControlPlugin">
@@ -294,6 +318,6 @@
         </scan>
         <range>
-          <min>0.120000</min>
-          <max>3.5</max>
+          <min>0.30000</min>
+          <max>5</max>
           <resolution>0.015000</resolution>
         </range>
@@ -445,3 +469,107 @@
     </sensor> -->
   </gazebo>
+  <joint name="gripper_extension" type="revolute">
+    <axis xyz="0 1 0"/>
+    <limit effort="50.0" lower="-1.57075" upper="0.2" velocity="0.5"/>
+    <origin rpy="0 0 0" xyz="0.05 0 0.1"/>
+    <parent link="base_link"/>
+    <child link="gripper_pole"/>
+  </joint>
+  <link name="gripper_pole">
+    <visual>
+      <geometry>
+        <cylinder length="0.1" radius="0.01"/>
+      </geometry>
+      <origin rpy="0 1.57075 0" xyz="0.1 0 0"/>
+    </visual>
+    <collision>
+      <origin rpy="0 1.57075 0" xyz="0.1 0 0"/>
+      <geometry>
+        <cylinder length="0.2" radius="0.01"/>
+      </geometry>
+    </collision>
+    <xacro:cylinder_inertia m="0.01" r="0.01" h="0.2"/>
+  </link>
+  <joint name="left_gripper_joint" type="prismatic">
+    <axis xyz="0 1 0"/>
+    <limit effort="100.0" lower="0.0" upper="0.06" velocity="0.25"/>
+    <origin rpy="0 0 0" xyz="0.2 0.01 0"/>
+    <parent link="gripper_pole"/>
+    <child link="left_gripper"/>
+  </joint>
+  <link name="left_gripper">
+    <visual>
+      <geometry>
+        <box size="0.1 0.02 0.02"/> <!-- Comprimento, largura, altura -->
+      </geometry>
+    </visual>
+    <collision>
+      <geometry>
+        <box size="0.1 0.02 0.02"/>
+      </geometry>
+    </collision>
+    <xacro:box_inertia m="0.015" w="0.02" h="0.02" d="0.1"/>
+  </link>
+  <joint name="left_tip_joint" type="fixed">
+    <origin rpy="0.0 0 0" xyz="0.06 0.001 0"/>
+    <parent link="left_gripper"/>
+    <child link="left_tip"/>
+  </joint>
+  <link name="left_tip">
+    <visual>
+      <origin rpy="0 0 -0.1" xyz="0.03 0 0"/>
+      <geometry>
+        <box size="0.06 0.01 0.01"/>
+      </geometry>
+    </visual>
+    <collision>
+      <origin rpy="0 0 -0.1" xyz="0.03 0 0"/>
+      <geometry>
+        <box size="0.06 0.01 0.01"/>
+      </geometry>
+    </collision>
+    <xacro:box_inertia m="0.005" w="0.01" h="0.01" d="0.06"/>
+  </link>
+  <joint name="right_gripper_joint" type="prismatic">
+    <axis xyz="0 1 0"/>
+    <limit effort="100.0" lower="-0.06" upper="0" velocity="0.25"/>
+    <origin rpy="0 0 0" xyz="0.2 -0.01 0"/>
+    <parent link="gripper_pole"/>
+    <child link="right_gripper"/>
+  </joint>
+  <link name="right_gripper">
+    <visual>
+      <origin rpy="-3.1415 0 0" xyz="0 0 0"/>
+      <geometry>
+        <box size="0.1 0.02 0.02"/>
+      </geometry>
+    </visual>
+    <collision>
+      <origin rpy="-3.1415 0 0" xyz="0 0 0"/>
+      <geometry>
+        <box size="0.1 0.02 0.02"/>
+      </geometry>
+    </collision>
+    <xacro:box_inertia m="0.015" w="0.02" h="0.02" d="0.1"/>
+  </link>
+  <joint name="right_tip_joint" type="fixed">
+    <origin rpy="-3.1415 0 0" xyz="0.06 -0.001 0"/>
+    <parent link="right_gripper"/>
+    <child link="right_tip"/>
+  </joint>
+  <link name="right_tip">
+    <visual>
+      <origin rpy="0 0 -0.1" xyz="0.03 0 0"/>
+      <geometry>
+        <box size="0.06 0.01 0.01"/>
+      </geometry>
+    </visual>
+    <collision>
+      <origin rpy="0 0 -0.1" xyz="0.03 0 0"/>
+      <geometry>
+        <box size="0.06 0.01 0.01"/>
+      </geometry>
+    </collision>
+    <xacro:box_inertia m="0.005" w="0.01" h="0.01" d="0.06"/>
+  </link>
 </robot>
